File: MCU_PCB.kicad_sch (KiCad schematic)
At the start: 0 parts

Commit message: V1
- Corrected SD-cards footprint and schematical represantation;
- Corrected RTC shematics:
	- changed oscilators power supply from internal 3v3 to Vbat so RTC works when PCB is disconnected from external power supply [PWR PCB];
	- 32 kHz to microcontroller now comes from RTC module;
	- added 100 nF decoupling capacitor to Vbat RTC pin.
- Corrected couple connections and component placement on PCB
Other:
- company: (none) -> BASEMENT
Changed lines of the file:
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@@
 (kicad_sch (version 20211123) (generator eeschema)
   (paper "A4")
+  (title_block
+    (date "%%date%%")
+    (rev "%%version%%")
+    (company "BASEMENT")
+  )
   (junction (at 144.78 116.84) (diameter 0) (color 0 0 0 0)
   )
@@
   )
   (symbol_instances
-    (path "/4b9b8940-4a19-4750-9b3b-069d0a42888c/3711eb2b-3d42-4440-a598-675f937f7b2d"
+    (path "/4b9b8940-4a19-4750-9b3b-069d0a42888c/e773b142-bf69-46b3-8dbc-a6f8018c1edc"
       (reference "#FLG0101") (unit 1) (value "PWR_FLAG") (footprint "")
     )
@@
       (reference "#FLG0103") (unit 1) (value "PWR_FLAG") (footprint "")
     )
+    (path "/d2da911f-3a7f-4dab-906d-6cdb198f9ff9/404492f4-38f2-4334-b705-62c4c7d3f9fb"
+      (reference "#FLG0104") (unit 1) (value "PWR_FLAG") (footprint "")
+    )
     (path "/2134c341-8583-49af-a415-faab632c4801/8fec2ae4-cb34-4b8b-b37b-c9ac8fc7ba16"
       (reference "#PWR01") (unit 1) (value "GND") (footprint "")
@@
       (reference "#PWR04") (unit 1) (value "GND") (footprint "")
     )
+    (path "/275a03c4-d5b5-4912-bf13-37b6cdfce08e/dcecd8a6-adf2-4555-9a11-4a269e2b96a7"
+      (reference "#PWR05") (unit 1) (value "GND") (footprint "")
+    )
     (path "/2134c341-8583-49af-a415-faab632c4801/29e3e138-9974-43b3-a805-23adacf1e90b"
       (reference "#PWR06") (unit 1) (value "+3.3V") (footprint "")
@@
       (reference "#PWR0110") (unit 1) (value "GND") (footprint "")
     )
-    (path "/275a03c4-d5b5-4912-bf13-37b6cdfce08e/a451ba0d-0017-4205-bad5-bd34a36b3975"
-      (reference "#PWR0111") (unit 1) (value "GND") (footprint "")
-    )
-    (path "/275a03c4-d5b5-4912-bf13-37b6cdfce08e/e3be8dea-9a7b-4b87-a14b-8f722357492d"
-      (reference "#PWR0112") (unit 1) (value "GND") (footprint "")
-    )
     (path "/275a03c4-d5b5-4912-bf13-37b6cdfce08e/5c60dcfc-07a4-4c7a-adee-751041a4f8ce"
       (reference "#PWR0113") (unit 1) (value "+3.3V") (footprint "")
@@
       (reference "#PWR0114") (unit 1) (value "GND") (footprint "")
     )
-    (path "/d2da911f-3a7f-4dab-906d-6cdb198f9ff9/3ad2cc9a-7d30-442b-b6a8-b936d95909f7"
+    (path "/d2da911f-3a7f-4dab-906d-6cdb198f9ff9/feaaaad4-551b-4e8e-9ff1-78cf2a4a3694"
       (reference "#PWR0115") (unit 1) (value "+BATT") (footprint "")
     )
@@
       (reference "#PWR0120") (unit 1) (value "GND") (footprint "")
     )
-    (path "/d2da911f-3a7f-4dab-906d-6cdb198f9ff9/a34290da-8f83-4dfa-b759-f5b1f2520c98"
-      (reference "#PWR0140") (unit 1) (value "+3.3V") (footprint "")
+    (path "/d2da911f-3a7f-4dab-906d-6cdb198f9ff9/2f71998d-0739-4971-9bfd-c11f827f3ca5"
+      (reference "#PWR0121") (unit 1) (value "+BATT") (footprint "")
+    )
+    (path "/d2da911f-3a7f-4dab-906d-6cdb198f9ff9/036ae249-cfd6-4913-94d6-83b865fc3f41"
+      (reference "#PWR0122") (unit 1) (value "GND") (footprint "")
     )
     (path "/5d39aa1b-6767-47e1-a0d3-ed950667e0c8/999c6a4f-503c-4d94-94a4-e36ff17a9fd0"
@@
       (reference "C4") (unit 1) (value "100nF") (footprint "Capacitor_SMD:C_0402_1005Metric")
     )
+    (path "/d2da911f-3a7f-4dab-906d-6cdb198f9ff9/45c2c467-b55f-4fd3-99b5-d85d70983cad"
+      (reference "C5") (unit 1) (value "100nF") (footprint "Capacitor_SMD:C_0402_1005Metric")
+    )
     (path "/2134c341-8583-49af-a415-faab632c4801/b6ad7a21-8c33-485c-9f13-87b73a644f97"
       (reference "C6") (unit 1) (value "100nF") (footprint "Capacitor_SMD:C_0402_1005Metric")
@@
       (reference "J3") (unit 1) (value "D2") (footprint "Connector_PinSocket_2.54mm:PinSocket_1x08_P2.54mm_Horizontal")
     )
-    (path "/275a03c4-d5b5-4912-bf13-37b6cdfce08e/80bc2490-8484-4540-a60c-a256d37810c3"
-      (reference "J4") (unit 1) (value "Micro_SD_Card") (footprint "footprints:Micro_SD")
+    (path "/275a03c4-d5b5-4912-bf13-37b6cdfce08e/58c2b9a7-4c62-43a6-be14-c32faf511b4d"
+      (reference "J4") (unit 1) (value "MEM2067-02-180-00-A_REVB") (footprint "footprints:GCT_MEM2067-02-180-00-A_REVB")
     )
     (path "/8d903d5a-c4b2-4966-809f-57caa871af62/bbc7b1e2-8d3f-43b8-a3fa-b64bb2786751"
@@
       (reference "U2") (unit 1) (value "MCP795W22-I/ST") (footprint "Package_SO:TSSOP-14_4.4x5mm_P0.65mm")
     )
-    (path "/2134c341-8583-49af-a415-faab632c4801/26c0282a-0831-4f40-af5f-11de8ca840da"
+    (path "/2134c341-8583-49af-a415-faab632c4801/28fbbe8a-5648-4b1a-843e-fee08dadd6f5"
       (reference "U3") (unit 1) (value "MC74AC138DR2G") (footprint "Package_SO:SOIC-16_3.9x9.9mm_P1.27mm")
     )
-    (path "/2134c341-8583-49af-a415-faab632c4801/c0730384-00b9-4fe1-baf3-9364d7c4f978"
+    (path "/2134c341-8583-49af-a415-faab632c4801/b81ba8ef-7507-4709-92a7-a05591bfe43c"
       (reference "U4") (unit 1) (value "MC74AC138DR2G") (footprint "Package_SO:SOIC-16_3.9x9.9mm_P1.27mm")
     )
-    (path "/5d39aa1b-6767-47e1-a0d3-ed950667e0c8/e4eb240c-0bb8-4bc8-809f-e871e4ec9258"
+    (path "/5d39aa1b-6767-47e1-a0d3-ed950667e0c8/fdbc7350-c5aa-43bc-aec8-6f058b887b62"
       (reference "U5") (unit 1) (value "ADT7310") (footprint "Package_SO:SOIC-8_3.9x4.9mm_P1.27mm")
     )
