File: SENS.kicad_sch (KiCad schematic)
At the start: 10 parts, among them U5 ADT7310, U6 LIS2MDLTR, U7 LSM6DSRX

Commit message: V1
- Corrected SD-cards footprint and schematical represantation;
- Corrected RTC shematics:
	- changed oscilators power supply from internal 3v3 to Vbat so RTC works when PCB is disconnected from external power supply [PWR PCB];
	- 32 kHz to microcontroller now comes from RTC module;
	- added 100 nF decoupling capacitor to Vbat RTC pin.
- Corrected couple connections and component placement on PCB
Other:
- company: (none) -> BASEMENT
Changed lines of the file:
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@@
 (kicad_sch (version 20211123) (generator eeschema)
   (paper "A4")
+  (title_block
+    (date "%%vdate%%")
+    (rev "%%version%%")
+    (company "BASEMENT")
+  )
   (junction (at 71.12 48.26) (diameter 0) (color 0 0 0 0)
   )
@@
     (pin "1")
   )
-  (symbol (lib_id "schematics:ADT7310") (at 40.64 88.9 0) (unit 1)
-    (in_bom yes) (on_board yes) (fields_autoplaced)
-    (property "Reference" "U5" (id 0) (at 40.64 71.12 0))
-    (property "Value" "ADT7310" (id 1) (at 40.64 73.66 0))
-    (property "Footprint" "Package_SO:SOIC-8_3.9x4.9mm_P1.27mm" (id 2) (at 40.64 71.12 0)
-      (effects (font (size 1.27 1.27)) hide)
-    )
-    (property "Datasheet" "" (id 3) (at 40.64 71.12 0)
-      (effects (font (size 1.27 1.27)) hide)
-    )
-    (pin "1")
-    (pin "2")
-    (pin "3")
-    (pin "4")
-    (pin "5")
-    (pin "6")
-    (pin "7")
-    (pin "8")
-  )
   (symbol (lib_id "Device:C_Small") (at 109.22 83.82 0) (unit 1)
     (in_bom yes) (on_board yes) (fields_autoplaced)
@@
     (pin "2")
   )
+  (symbol (lib_id "schematics:ADT7310") (at 40.64 88.9 0) (unit 1)
+    (in_bom yes) (on_board yes) (fields_autoplaced)
+    (property "Reference" "U5" (id 0) (at 40.64 71.12 0))
+    (property "Value" "ADT7310" (id 1) (at 40.64 73.66 0))
+    (property "Footprint" "Package_SO:SOIC-8_3.9x4.9mm_P1.27mm" (id 2) (at 40.64 71.12 0)
+      (effects (font (size 1.27 1.27)) hide)
+    )
+    (property "Datasheet" "" (id 3) (at 40.64 71.12 0)
+      (effects (font (size 1.27 1.27)) hide)
+    )
+    (pin "1")
+    (pin "2")
+    (pin "3")
+    (pin "4")
+    (pin "5")
+    (pin "6")
+    (pin "7")
+    (pin "8")
+  )
 )
